File: fridge-beeper/schematic/fridge-beeper.kicad_sch (KiCad schematic)
At the start: 5 parts, among them SW1 Door Sensor, SW2 SW_SPST, U1 ATtiny13A-P

Commit message: Add boost converter to schematic
Parts:
- removed SW2: SW_SPST, symbol Switch:SW_SPST
Other:
- note added: "3V3 SMPS"
- note removed: "Battery Holder"
Changed lines of the file:
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@@
 	)
 	(rectangle
-		(start 54.61 53.34)
-		(end 74.93 80.01)
+		(start 57.15 55.88)
+		(end 67.31 66.04)
 		(stroke
 			(width 0)
@@
 		)
 	)
-	(text "Battery Holder"
-		(exclude_from_sim no)
-		(at 46.736 54.356 0)
+	(text "3V3 SMPS"
+		(exclude_from_sim no)
+		(at 62.23 60.96 0)
 		(effects
 			(font
@@
 					(unit 1)
 				)
-			)
-		)
-	)
-	(symbol
-		(lib_id "Switch:SW_SPST")
-		(at 62.23 60.96 90)
-		(unit 1)
-		(exclude_from_sim no)
-		(in_bom yes)
-		(on_board yes)
-		(dnp no)
-		(property "Reference" "SW2"
-			(at 58.674 60.96 0)
-			(effects
-				(font
-					(size 1.27 1.27)
-				)
-			)
-		)
-		(property "Value" "SW_SPST"
-			(at 58.42 60.96 0)
-			(effects
-				(font
-					(size 1.27 1.27)
-				)
-				(hide yes)
-			)
-		)
-		(property "Footprint" ""
-			(at 62.23 60.96 0)
-			(effects
-				(font
-					(size 1.27 1.27)
-				)
-				(hide yes)
-			)
-		)
-		(property "Datasheet" "~"
-			(at 62.23 60.96 0)
-			(effects
-				(font
-					(size 1.27 1.27)
-				)
-				(hide yes)
-			)
-		)
-		(property "Description" "Single Pole Single Throw (SPST) switch"
-			(at 62.23 60.96 0)
-			(effects
-				(font
-					(size 1.27 1.27)
-				)
-				(hide yes)
-			)
-		)
-		(pin "1"
-		)
-		(pin "2"
-		)
-		(instances
-			(project ""
-				(path "/8f58275b-bc43-493f-8ccf-458b2bd48b80"
-					(reference "SW2")
-					(unit 1)
-				)
